Commit message: Revert "modificações"
This reverts commit b85e7e3d35631f79ecc29f74505ba941386a34e0, reversing
changes made to 0cae5f8f725d271470a87959a19c4259d5f7e5df.

File: urdf/_d435.urdf.xacro (robot description, xacro)
@@ -8,5 +8,5 @@
 <robot name="sensor_d435" xmlns:xacro="http://ros.org/wiki/xacro">
   <!--File includes-->
-  <xacro:include filename="$(find ggcnn_pkg)/urdf/_d435.gazebo.xacro"/>
+  <xacro:include filename="$(find trajectory_pkg)/urdf/_d435.gazebo.xacro"/>
   <xacro:macro name="sensor_d435" params="name:=camera topics_ns:=camera parent *origin publish_pointcloud:=true">
     <xacro:property name="M_PI" value="3.1415926535897931" />

File: urdf/ur5_gripper_cam.xacro (robot description, xacro)
@@ -52,7 +52,7 @@
   -->
     <!-- include the camera realsense2 d_435 -->
-    <xacro:include filename="$(find ggcnn_pkg)/urdf/_d435.urdf.xacro" />
+    <xacro:include filename="$(find trajectory_pkg)/urdf/_d435.urdf.xacro" />
     <!-- include the gripper -->
-    <xacro:include filename="$(find ggcnn_pkg)/urdf/eef.xacro"/>
+    <xacro:include filename="$(find trajectory_pkg)/urdf/eef.xacro"/>
     <transmission name="shoulder_pan_trans">
         <type>transmission_interface/SimpleTransmission</type>
@@ -378,5 +378,5 @@
       <origin xyz="0 0 0" rpy="0 0 0"/>
       <geometry>
-        <mesh filename="package://ggcnn_pkg/models/cam_support/CAM_support.STL" scale="0.001 0.001 0.001"/>
+        <mesh filename="package://trajectory_pkg/models/cam_support/CAM_support.STL" scale="0.001 0.001 0.001"/>
       </geometry>
     </collision>
@@ -385,5 +385,5 @@
       <origin rpy="${1.57 - 0.244} ${3.14} -1.57" xyz="${0.002 - 0.03 + 0.023} ${-0.023 + 0.03 - 0.01} ${0.13915-0.205-0.092}"/>
       <geometry>
-        <mesh filename="package://ggcnn_pkg/models/cam_support/CAM_support.STL" scale="0.001 0.001 0.001"/>
+        <mesh filename="package://trajectory_pkg/models/cam_support/CAM_support.STL" scale="0.001 0.001 0.001"/>
       </geometry>
       <material name="Cyan">

File: urdf/ur5_gripper_cam_2.xacro (robot description, xacro)
@@ -51,6 +51,6 @@
           this location. Nor can they rely on the existence of the macro.
   -->
-    <xacro:include filename="$(find ggcnn_pkg)/urdf/eef.xacro"/>
-    <xacro:include filename="$(find ggcnn_pkg)/urdf/_d435.urdf.xacro" />
+    <xacro:include filename="$(find trajectory_pkg)/urdf/eef.xacro"/>
+    <xacro:include filename="$(find trajectory_pkg)/urdf/_d435.urdf.xacro" />
     <transmission name="shoulder_pan_trans">
         <type>transmission_interface/SimpleTransmission</type>
@@ -376,5 +376,5 @@
       <origin xyz="0 0 0" rpy="0 0 0"/>
       <geometry>
-        <mesh filename="package://ggcnn_pkg/models/cam_support/CAM_support.STL" scale="0.001 0.001 0.001"/>
+        <mesh filename="package://trajectory_pkg/models/cam_support/CAM_support.STL" scale="0.001 0.001 0.001"/>
       </geometry>
     </collision>
@@ -383,5 +383,5 @@
       <origin rpy="${1.57 - 0.244} ${3.14} -1.57" xyz="${0.002 - 0.03 + 0.023} ${-0.023 + 0.03 - 0.01} ${0.13915-0.205-0.092}"/>
       <geometry>
-        <mesh filename="package://ggcnn_pkg/models/cam_support/CAM_support.STL" scale="0.001 0.001 0.001"/>
+        <mesh filename="package://trajectory_pkg/models/cam_support/CAM_support.STL" scale="0.001 0.001 0.001"/>
       </geometry>
       <material name="Cyan">

File: urdf/ur5_gripper_cam_racunho.xacro (robot description, xacro)
@@ -72,5 +72,5 @@
       <origin xyz="0 0 0" rpy="0 0 0"/>
       <geometry>
-        <mesh filename="package://ggcnn_pkg/models/cam_support/CAM_support.STL" scale="0.001 0.001 0.001"/>
+        <mesh filename="package://trajectory_pkg/models/cam_support/CAM_support.STL" scale="0.001 0.001 0.001"/>
       </geometry>
     </collision>
@@ -79,5 +79,5 @@
       <origin rpy="${1.57 - 0.244} ${3.14} -1.57" xyz="${0.002 - 0.03 + 0.023} ${-0.023 + 0.03 - 0.01} ${0.13915-0.205-0.092}"/>
       <geometry>
-        <mesh filename="package://ggcnn_pkg/models/cam_support/CAM_support.STL" scale="0.001 0.001 0.001"/>
+        <mesh filename="package://trajectory_pkg/models/cam_support/CAM_support.STL" scale="0.001 0.001 0.001"/>
       </geometry>
       <material name="Cyan">
@@ -140,5 +140,5 @@
 <!-- *************************************************************** -->
     <!-- include the gripper -->
-    <xacro:include filename="$(find ggcnn_pkg)/urdf/eef.xacro"/>
+    <xacro:include filename="$(find trajectory_pkg)/urdf/eef.xacro"/>
     <transmission name="shoulder_pan_trans">
         <type>transmission_interface/SimpleTransmission</type>

File: urdf/ur5_traj_gripper.xacro (robot description, xacro)
@@ -51,5 +51,5 @@
           this location. Nor can they rely on the existence of the macro.
   -->
-    <xacro:include filename="$(find ggcnn_pkg)/urdf/eef.xacro"/>
+    <xacro:include filename="$(find trajectory_pkg)/urdf/eef.xacro"/>
     <transmission name="shoulder_pan_trans">
         <type>transmission_interface/SimpleTransmission</type>
